File: sds_tool/sds_tool.sch (KiCad schematic (older format))
At the start: 17 parts, among them P1 CONN_01X06, Q1 MMBT3904, Q2 MMBT3904, Q3 MMBT3904, Q4 MMBT3904, Q5 MMBT3904, Q6 MMBT3904, U1 Teensy2.0, U2 STl9637

Commit message: Fix value of R4
Parts:
- R4: value 630 -> 820
Changed lines of the file:
@@
 P 7300 1450
 F 0 "R4" V 7380 1450 50  0000 C CNN
-F 1 "630" V 7300 1450 50  0000 C CNN
+F 1 "820" V 7300 1450 50  0000 C CNN
 F 2 "Resistors_SMD:R_0805_HandSoldering" V 7230 1450 50  0001 C CNN
 F 3 "" H 7300 1450 50  0000 C CNN
